File: fanboard.kicad_pcb (KiCad board)
At the start: 2 copper layers, 48 x 32 mm, 36 parts, among them J1 HLE-103-02-S-DV-LC, J2 TC2050-IDC-NL-FP, J3 TC2050-IDC-NL-FP, J4 78171-0004, Q1 NVJD4401N, SW1 CVS-03B, U1 TVS3301DRBR, U2 TPS26624DRCR, U3 LMZM23600V3SILR, U4 CC3235MODASF12MONR

Commit message: Update to KiCad 6; add additional manufacturer STEP files.
Other:
- net class Default removed
- net class Power removed
